File: Adlib.kicad_pcb (KiCad board)
At the start: 2 copper layers, 135.3 x 106.7 mm, 61 parts, among them J1 CONN_01X05, P1 IRQ, P2 ADDR, Q1 2N3904, U1 74LS109, U2 74LS138, U3 74LS138, U4 74LS245, U5 74LS04, U6 YM3812, U7 YM3014B, U8 RC4136, U9 LM386N

Commit message: Add files via upload
Parts:
- added G***: LOGO, Battery:AdLib_logo, F.Cu at (81.9, 75.9)
Connections:
- net /~IOR renamed /~{IOR}
- net /~IOW renamed /~{IOW}
- net /~IRQ renamed /~{IRQ}
- net /~READ renamed /~{READ}
- net /~RESET renamed /~{RESET}
- net /~WRITE renamed /~{WRITE}
Routing:
- net (no net): track 0.00 -> 113.3 mm
- net GND: track 316.4 -> 318.1 mm
Other:
- net class Default removed
- board text added: "R"
- board text removed: "1"
- board text removed: "2"
- board text removed: "3"
- board text removed: "31"
- board text removed: "5"
- board text removed: "A"
- board text removed: "B"
- board text removed: "C"
- board text removed: "D"
- board text removed: "Replica of 1990 Ad Lib"
